File: PCB/Smarttree_CMU_5.2.3.brd (EAGLE design)
At the start: 104.9 x 78.1 mm, 100 parts

Commit message: comments about changes
Parts:
- removed C21, C22: (no value), standardparts:0805
- removed C27, C34, C35, C36, C37: 0.1uF, SparkFun:0603-CAP
- removed C29: (no value), SparkFun:0603-CAP
- removed FAN1: DCJ0202, con-jack:DCJ0202
- removed JP1, JP2: (no value), SparkFun-Connectors:1X06_LONGPADS
- removed JP3: (no value), SparkFun-Connectors:1X08_LONGPADS
- removed JP5: comm-due, SparkFun-Connectors:1X08_LONGPADS
- removed JP6: (no value), SparkFun:1X06_LONGPADS
- removed Q1: (no value), adafruit:SOT23
- removed R5: 330, adafruit:R0805
- removed R6: 10k, adafruit:R0805
- removed U$2: ADR366B-SOT23, Francis-Project:SOT23-5
- removed U$3: MAX3222, Francis-Project:SO18
- removed X1: (no value), SparkFun-Connectors:DB9
- moved C23 28.4 mm to (49.5, 9.91)
- moved C24 28.4 mm to (53.8, 9.91)
- moved C28 28.4 mm to (78.0, 43.4)
- moved C7 28.4 mm to (58.4, 48.0)
- moved CMU4 28.4 mm to (15.7, 47.2)
- moved R17 28.4 mm to (41.9, 42.9)
- moved R25 28.4 mm to (40.9, 30.2)
- moved ANALOG_MUX 28.4 mm to (40.1, 17.5)
- moved C25 28.4 mm to (49.9, 21.6)
- moved C31 28.4 mm to (56.5, 21.6)
- moved C32 28.4 mm to (46.4, 21.6)
- moved D2 28.4 mm to (69.8, 17.9)
- moved F2 28.4 mm to (63.9, 17.9)
- moved LED1 28.4 mm to (63.5, 7.62)
- moved LMT87 28.4 mm to (53.1, 5.33)
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Connections:
- removed net N$1: FAN1.2, FAN1.3, Q1.3
- removed net N$10: C35.1, U$3.7
- removed net N$11: C27.1, U$3.2
- removed net N$12: C29.1, Q1.1, R5.1, R6.1
- removed net N$21: C27.2, U$3.4
- removed net N$22: C34.1, U$3.5
- removed net N$23: C34.2, U$3.6
- removed net N$25: C36.2, U$3.3
- removed net N$27: U$3.15, X1.2
- removed net N$29: U$3.14, X1.3
- removed net N$31: JP1.6, JP2.6
- removed net RFAN: R5.2, U$1.13
- removed net RX3: JP5.7
- removed net SCL: JP5.1
- removed net SDA: JP5.2
- removed net TX2: JP5.6
- removed net VDD: C37.2, JP1.5, JP2.5, U$3.17
- removed net VIN: JP1.1, JP2.1, X1.4, X1.8
- removed net VREF: C21.1, U$1.AREF, U$2.4
- net 12V: no longer FAN1.1
- net 5V: no longer C22.2, JP1.4, JP2.4, U$2.3
- net GND: no longer C21.2, C22.1, C29.2, C35.2, C36.1, C37.1, JP1.2, JP1.3, JP2.2, JP2.3, Q1.2, R6.2, U$2.2, U$3.1, U$3.11, U$3.16, U$3.9, X1.5, X1.9
- net N$2: no longer JP5.5
- net RX1: no longer JP5.3, U$3.13
- net SHDN: no longer JP5.8, U$3.18
- net TX1: no longer JP5.4, U$3.12
Routing:
- net VDD: track 89.6 -> 0.00 mm, vias 1 -> 0
- net N$29: track 51.4 -> 0.00 mm, vias 1 -> 0
- net N$27: track 51.1 -> 0.00 mm, vias 1 -> 0
- net RFAN: track 41.1 -> 0.00 mm
- net VIN: track 34.3 -> 0.00 mm
- net VREF: track 27.8 -> 0.00 mm
- net SHDN: track 46.2 -> 19.1 mm, vias 1 -> 0
- net RX1: track 53.5 -> 38.3 mm, vias 1 -> 0
- net TX1: track 36.9 -> 22.2 mm, vias 2 -> 1
- net GND: track 107.4 -> 94.8 mm, vias 14 -> 11
- net N$12: track 10.6 -> 0.00 mm
- net N$1: track 9.39 -> 0.00 mm
- net N$11: track 8.88 -> 0.00 mm, vias 2 -> 0
- net N$31: track 8.26 -> 0.00 mm
- net 5V: track 14.6 -> 6.35 mm
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Other:
- board size 104.9 x 78.1 mm -> 88.4 x 55 mm
- board text added: "----Layout ->make it nicer ->put analog MUX on the top layer ->make a debugging interface for sensor reading ->switch bypass with jumper ->make sensor board connectors closer to the edge"
- board text removed: "ESW"
- board text removed: "NU"
- board text removed: "SmartTree"

Commit message: bms cnt'd
Routing:
- net 12V: track 99.0 -> 82.1 mm
- net GND: track 94.8 -> 80.9 mm
Changed lines of the file:
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@@
 <contactref element="C24" pad="2"/>
 <contactref element="C23" pad="2"/>
-<wire x1="19.558" y1="31.75" x2="20.574" y2="30.734" width="0.3048" layer="1"/>
-<wire x1="22.098" y1="30.734" x2="22.606" y2="31.242" width="0.3048" layer="1"/>
-<wire x1="22.606" y1="31.242" x2="23.114" y2="30.734" width="0.3048" layer="1"/>
-<wire x1="23.114" y1="30.734" x2="25.146" y2="30.734" width="0.3048" layer="1"/>
-<wire x1="25.146" y1="30.734" x2="25.654" y2="31.242" width="0.3048" layer="1"/>
+<wire x1="19.558" y1="31.75" x2="20.574" y2="30.734" width="0" layer="19" extent="1-16"/>
+<wire x1="22.098" y1="30.734" x2="22.606" y2="31.242" width="0" layer="19" extent="1-16"/>
+<wire x1="22.606" y1="31.242" x2="23.114" y2="30.734" width="0" layer="19" extent="1-16"/>
+<wire x1="23.114" y1="30.734" x2="25.146" y2="30.734" width="0" layer="19" extent="1-16"/>
+<wire x1="25.146" y1="30.734" x2="25.654" y2="31.242" width="0" layer="19" extent="1-16"/>
 <contactref element="C31" pad="2"/>
 <contactref element="C32" pad="1"/>
@@
 <wire x1="58.039" y1="23.876" x2="57.785" y2="24.3078" width="0.254" layer="1"/>
 <wire x1="61.148" y1="10.16" x2="63.312" y2="10.16" width="0.254" layer="1"/>
-<wire x1="22.098" y1="30.734" x2="20.574" y2="30.734" width="0.3048" layer="1"/>
-<wire x1="20.574" y1="30.734" x2="18.542" y2="28.702" width="0.3048" layer="1"/>
-<wire x1="18.542" y1="28.702" x2="18.542" y2="24.768" width="0.3048" layer="1"/>
+<wire x1="22.098" y1="30.734" x2="20.574" y2="30.734" width="0" layer="19" extent="1-16"/>
+<wire x1="20.574" y1="30.734" x2="18.542" y2="28.702" width="0" layer="19" extent="1-16"/>
+<wire x1="18.542" y1="28.702" x2="18.542" y2="24.768" width="0" layer="19" extent="1-16"/>
 <wire x1="21.8694" y1="20.7264" x2="21.8694" y2="23.3426" width="0.3048" layer="1"/>
 <wire x1="21.8694" y1="23.3426" x2="20.574" y2="24.638" width="0.3048" layer="1"/>
@@
 <wire x1="19.189" y1="16.51" x2="19.189" y2="21.321" width="0.635" layer="1"/>
 <wire x1="19.189" y1="21.321" x2="18.542" y2="21.968" width="0.635" layer="1"/>
-<wire x1="18.542" y1="21.968" x2="15.878" y2="21.968" width="0.635" layer="1"/>
-<wire x1="15.878" y1="21.968" x2="13.97" y2="23.876" width="0.635" layer="1"/>
-<wire x1="13.97" y1="23.876" x2="13.97" y2="35.358" width="0.635" layer="1"/>
 <wire x1="26.4414" y1="20.7264" x2="26.4414" y2="19.0754" width="0.635" layer="1"/>
 <wire x1="26.4414" y1="19.0754" x2="25.4" y2="18.034" width="0.635" layer="1"/>
