File: PCB/Smarttree_CMU_5.2.3.sch (EAGLE design)
At the start: 100 parts

Commit message: comments about changes
Parts:
- removed C21, C22: (no value), standardparts:CAPACITOR.0805
- removed C27, C34, C35, C36, C37: 0.1uF, SparkFun:CAP0603-CAP
- removed C29: (no value), SparkFun:CAP0603-CAP
- removed FAN1: DCJ0202, con-jack:DCJ0202
- removed JP1, JP2: (no value), SparkFun-Connectors:M06LONGPADS
- removed JP3: (no value), SparkFun-Connectors:M08LONGPADS
- removed JP5: comm-due, SparkFun-Connectors:M08LONGPADS
- removed JP6: (no value), SparkFun:M06LONGPADS
- removed Q1: (no value), adafruit:MOSFET-NREFLOW
- removed R5: 330, adafruit:R-US_R0805
- removed R6: 10k, adafruit:R-US_R0805
- removed U$2: ADR366B-SOT23, Francis-Project:ADR366B-SOT23
- removed U$3: MAX3222, Francis-Project:MAX3222
- removed X1: (no value), SparkFun-Connectors:DB9FEMALE
Connections:
- removed net N$1: FAN1.2, FAN1.3, Q1.D
- removed net N$10: C35.1, U$3G$1.V-
- removed net N$11: C27.1, U$3G$1.C1+
- removed net N$12: C29.1, Q1.G, R5.1, R6.1
- removed net N$21: C27.2, U$3G$1.C1-
- removed net N$22: C34.1, U$3G$1.C2+
- removed net N$23: C34.2, U$3G$1.C2-
- removed net N$25: C36.2, U$3G$1.V+
- removed net N$27: U$3G$1.T1OUT, X1.2
- removed net N$29: U$3G$1.R1IN, X1.3
- removed net N$31: JP1.6, JP2.6
- removed net RFAN: R5.2, U$1.13
- removed net RX3: JP5.7
- removed net SCL: JP5.1
- removed net SDA: JP5.2
- removed net TX2: JP5.6
- removed net VDD: C37.2, JP1.5, JP2.5, U$3G$2.VCC
- removed net VIN: JP1.1, JP2.1, X1.4, X1.8
- removed net VREF: C21.1, U$1.AREF, U$2.OUT
- net 12V: no longer FAN1.1
- net 5V: no longer C22.2, JP1.4, JP2.4, U$2.VIN
- net GND: no longer C21.2, C22.1, C29.2, C35.2, C36.1, C37.1, JP1.2, JP1.3, JP2.2, JP2.3, Q1.S, R6.2, U$2.GND, U$3G$1.EN/, U$3G$1.R2IN, U$3G$1.T2IN, U$3G$2.GND, X1.5, X1.9
- net N$2: no longer JP5.5
- net RX1: no longer JP5.3, U$3G$1.R1OUT
- net SHDN: no longer JP5.8, U$3G$1.SHDN/
- net TX1: no longer JP5.4, U$3G$1.T1IN
Other:
- note added: "----Schematic ->RS-232 direct mapping (w/o adapter) ->Software reset for each sensor board ->9 to 3V3 regulator on the board ->get rid of 3v3 ref pin (VREF)"

Commit message: bms cnt'd
Other:
- note added: "----Schematic ->RS-232 direct mapping (w/o adapter) ->Software reset for each sensor board ->9 to 3V3 regulator on the board ->get rid of 3v3 ref pin (VREF) ->isolate arduino power"
- note removed: "----Schematic ->RS-232 direct mapping (w/o adapter) ->Software reset for each sensor board ->9 to 3V3 regulator on the board ->get rid of 3v3 ref pin (VREF)"
- moved on the sheet: 5V_REG, C10, C6
Changed lines of the file:
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@@
 -&gt;9 to 3V3 regulator on the board
 -&gt;get rid of 3v3 ref pin (VREF)
-</text>
+-&gt;isolate arduino power</text>
 </plain>
 <instances>
 <instance part="VDD2" gate="G$1" x="127" y="147.32"/>
-<instance part="VDD5" gate="G$1" x="210.82" y="111.76"/>
-<instance part="SUPPLY19" gate="GND" x="228.6" y="81.28"/>
-<instance part="5V" gate="G$1" x="243.84" y="109.22"/>
+<instance part="VDD5" gate="G$1" x="213.36" y="129.54"/>
+<instance part="SUPPLY19" gate="GND" x="231.14" y="99.06"/>
+<instance part="5V" gate="G$1" x="246.38" y="127"/>
 <instance part="SUPPLY10" gate="GND" x="109.22" y="116.84"/>
-<instance part="5V_REG" gate="G$1" x="228.6" y="104.14"/>
-<instance part="C10" gate="G$1" x="210.82" y="96.52">
-<attribute name="OC_NEWARK" x="210.82" y="96.52" size="1.778" layer="96" display="off"/>
-<attribute name="MF" x="210.82" y="96.52" size="1.778" layer="96" display="off"/>
-<attribute name="MPN" x="210.82" y="96.52" size="1.778" layer="96" display="off"/>
-</instance>
-<instance part="C6" gate="G$1" x="243.84" y="96.52">
-<attribute name="OC_NEWARK" x="243.84" y="96.52" size="1.778" layer="96" display="off"/>
-<attribute name="MF" x="243.84" y="96.52" size="1.778" layer="96" display="off"/>
-<attribute name="MPN" x="243.84" y="96.52" size="1.778" layer="96" display="off"/>
+<instance part="5V_REG" gate="G$1" x="231.14" y="121.92"/>
+<instance part="C10" gate="G$1" x="213.36" y="114.3">
+<attribute name="OC_NEWARK" x="213.36" y="114.3" size="1.778" layer="96" display="off"/>
+<attribute name="MF" x="213.36" y="114.3" size="1.778" layer="96" display="off"/>
+<attribute name="MPN" x="213.36" y="114.3" size="1.778" layer="96" display="off"/>
+</instance>
+<instance part="C6" gate="G$1" x="246.38" y="114.3">
+<attribute name="OC_NEWARK" x="246.38" y="114.3" size="1.778" layer="96" display="off"/>
+<attribute name="MF" x="246.38" y="114.3" size="1.778" layer="96" display="off"/>
+<attribute name="MPN" x="246.38" y="114.3" size="1.778" layer="96" display="off"/>
 </instance>
 <instance part="D1" gate="G$1" x="104.14" y="134.62" rot="R180">
@@
 <net name="GND" class="0">
 <segment>
-<wire x1="243.84" y1="88.9" x2="228.6" y2="88.9" width="0.1524" layer="91"/>
+<wire x1="246.38" y1="106.68" x2="231.14" y2="106.68" width="0.1524" layer="91"/>
 <pinref part="5V_REG" gate="G$1" pin="GND"/>
-<wire x1="228.6" y1="88.9" x2="210.82" y2="88.9" width="0.1524" layer="91"/>
-<wire x1="228.6" y1="91.44" x2="228.6" y2="88.9" width="0.1524" layer="91"/>
-<junction x="228.6" y="88.9"/>
+<wire x1="231.14" y1="106.68" x2="213.36" y2="106.68" width="0.1524" layer="91"/>
+<wire x1="231.14" y1="109.22" x2="231.14" y2="106.68" width="0.1524" layer="91"/>
+<junction x="231.14" y="106.68"/>
 <pinref part="SUPPLY19" gate="GND" pin="GND"/>
-<wire x1="228.6" y1="88.9" x2="228.6" y2="83.82" width="0.1524" layer="91"/>
+<wire x1="231.14" y1="106.68" x2="231.14" y2="101.6" width="0.1524" layer="91"/>
 <pinref part="C10" gate="G$1" pin="-"/>
-<wire x1="210.82" y1="88.9" x2="210.82" y2="91.44" width="0.1524" layer="91"/>
+<wire x1="213.36" y1="106.68" x2="213.36" y2="109.22" width="0.1524" layer="91"/>
 <pinref part="C6" gate="G$1" pin="-"/>
-<wire x1="243.84" y1="88.9" x2="243.84" y2="91.44" width="0.1524" layer="91"/>
+<wire x1="246.38" y1="106.68" x2="246.38" y2="109.22" width="0.1524" layer="91"/>
 </segment>
 <segment>
@@
 <pinref part="5V" gate="G$1" pin="5V"/>
 <pinref part="5V_REG" gate="G$1" pin="VOUT"/>
-<wire x1="243.84" y1="104.14" x2="243.84" y2="109.22" width="0.1524" layer="91"/>
-<wire x1="241.3" y1="104.14" x2="243.84" y2="104.14" width="0.1524" layer="91"/>
+<wire x1="246.38" y1="121.92" x2="246.38" y2="127" width="0.1524" layer="91"/>
+<wire x1="243.84" y1="121.92" x2="246.38" y2="121.92" width="0.1524" layer="91"/>
 <pinref part="C6" gate="G$1" pin="+"/>
-<wire x1="243.84" y1="104.14" x2="243.84" y2="99.06" width="0.1524" layer="91"/>
-<junction x="243.84" y="104.14"/>
+<wire x1="246.38" y1="121.92" x2="246.38" y2="116.84" width="0.1524" layer="91"/>
+<junction x="246.38" y="121.92"/>
 </segment>
 <segment>
@@
 <segment>
 <pinref part="VDD5" gate="G$1" pin="12V"/>
-<wire x1="210.82" y1="109.22" x2="210.82" y2="104.14" width="0.1524" layer="91"/>
+<wire x1="213.36" y1="127" x2="213.36" y2="121.92" width="0.1524" layer="91"/>
 <pinref part="5V_REG" gate="G$1" pin="VIN"/>
-<wire x1="215.9" y1="104.14" x2="210.82" y2="104.14" width="0.1524" layer="91"/>
+<wire x1="218.44" y1="121.92" x2="213.36" y2="121.92" width="0.1524" layer="91"/>
 <pinref part="C10" gate="G$1" pin="+"/>
-<wire x1="210.82" y1="99.06" x2="210.82" y2="104.14" width="0.1524" layer="91"/>
-<junction x="210.82" y="104.14"/>
-</segment>
-<segment>
+<wire x1="213.36" y1="116.84" x2="213.36" y2="121.92" width="0.1524" layer="91"/>
+<junction x="213.36" y="121.92"/>
+</segment>
+<segment>
