File: PCB/Smarttree_BMS_3.2.brd (EAGLE design)
At the start: 66.1 x 45.9 mm, 41 parts, among them X2 057-006-0

Commit message: new cmu pcb
Parts:
- removed C10, C3: 4.7nF, adafruit:C0805
- removed C7, C9: 47nF, adafruit:C0805
- removed LM1117: LM2937_SOT223, linear2:SOT223
- removed U$1, U$4: HMS-5P-SOTA, Francis-Project:SMD_CURR_SENSE
- removed U$6: S22P015S05, Allen:S22P015S05
- added CS1, CS2: S22P015S05, Allen:S22P015S05
- added R10, R11: 1k, adafruit:R0805
- added R12, R9: 10k, adafruit:R0805
- added R13, R14: 100, adafruit:R0805
- added Z1, Z2: (no value), SparkFun:SOD-323
- C1, C2: value 47nF -> 0.1uF
- C5: device SparkFun-Retired:EIA3216 -> adafruit:C0805
- C6: value 10uF -> 0.1uF; device SparkFun-Retired:EIA3216 -> adafruit:C0805
- moved C5 35.2 mm to (62.2, 35.6), turned to 90 degrees
- moved LMT87 21.1 mm to (37.0, 22.2)
- moved C4 20.6 mm to (34.0, 19.8), flipped to the top, turned to 270 degrees
- moved C8 19.8 mm to (36.8, 19.8), flipped to the top, turned to 270 degrees
- moved C2 13.8 mm to (30.0, 32.8), turned to 0 degrees
- moved R7 10.7 mm to (60.2, 41.9), flipped to the top, turned to 90 degrees
- moved C1 8.67 mm to (20.1, 35.6), turned to 270 degrees
- moved R8 8.32 mm to (57.7, 41.9), flipped to the top, turned to 90 degrees
- moved Q3 8.05 mm to (12.2, 41.8), flipped to the top, turned to 90 degrees
- moved R3 7.25 mm to (18.7, 41.9), flipped to the top, turned to 90 degrees
- moved Q4 7.06 mm to (53.8, 41.9), flipped to the top, turned to 90 degrees
- moved R5 5.98 mm to (48.3, 40.6), turned to 180 degrees
- moved R4 5.95 mm to (16.0, 41.9), flipped to the top, turned to 90 degrees
- moved C6 5.74 mm to (40.1, 32.8), turned to 180 degrees
- moved X2 5.68 mm to (32.0, 43.2)
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Connections:
- removed net 2.5V: C2.1, C6.A, C9.1, LM1117.3, U$1.VREF, U$4.VREF
- new net N$12: CS1.7, R11.1, R9.2
- new net N$13: CS2.7, R10.2, R12.1
- new net N$14: R14.2, Z1.1
- new net N$9: R13.2, Z2.1
- net ARR_CURR+: now also CS2.4, CS2.5, CS2.6; no longer U$1.I-
- net ARR_CURR-: now also CS2.1, CS2.2, CS2.3; no longer U$1.I+
- net BAT_CURR+: now also CS1.4, CS1.5, CS1.6; no longer U$4.I-
- net BAT_CURR-: now also CS1.1, CS1.2, CS1.3; no longer U$4.I+
- net CSI: now also C2.1, R12.2, R13.1; no longer C10.1, U$4.OUTPUT
- net CSO: now also C6.1, R11.2, R14.1; no longer C3.1, U$1.OUTPUT
- net GND: now also C5.2, C6.2, CS1.8, CS2.8, R10.1, R9.1, Z1.2, Z2.2; no longer C10.2, C3.2, C5.C, C6.C, C7.2, C9.2, LM1117.2, LM1117.4, U$1.GND, U$4.GND
- net VCC: now also C5.1, CS1.9, CS2.9; no longer C5.A, C7.1, LM1117.1, U$1.VCC, U$4.VCC
Routing:
- net 2.5V: track 82.9 -> 0.00 mm
- net RELAY_OUT: track 15.9 -> 38.8 mm
- net VCC: track 16.5 -> 0.00 mm
- net CSO: track 42.8 -> 27.2 mm
- net RELAY_IN: track 31.7 -> 16.8 mm, vias 1 -> 0
- net GND: track 51.8 -> 43.3 mm, vias 5 -> 6
- net BAT_CURR-: track 7.47 -> 15.4 mm
- net N$12: track 0.00 -> 7.34 mm
- net N$13: track 0.00 -> 6.80 mm
- net BAT_GND: track 58.9 -> 52.6 mm
- net N$5: track 7.48 -> 2.46 mm
- net ARR+: track 20.0 -> 15.8 mm
- net ARR_CURR-: track 12.4 -> 16.2 mm
- net CSI: track 29.8 -> 26.0 mm, vias 0 -> 1
- net N$4: track 4.32 -> 7.89 mm
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Other:
- board size 66.1 x 45.9 mm -> 67.4 x 45.9 mm
- board text added: "/Users/chentuofei/Desktop/ME433/HW2/wildbw.bmp"
- board text added: "SmartTree CMU 3.3"
