File: PCB/Smarttree_CMU_4.sch (EAGLE design)
At the start: 43 parts, among them X2 057-006-0

Commit message: gerber file and finalized cmu design
Parts:
- removed VS_JMP-: (no value), SparkFun:M02
- added JP1: M01OFFSET, SparkFun:M01OFFSET
Connections:
- net BAT_GND: now also JP1.1; no longer VS_JMP-.1, VS_JMP-.2
Changed lines of the file:
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@@
 <setting verticaltext="up"/>
 </settings>
-<grid distance="0.1" unitdist="inch" unit="inch" style="lines" multiple="1" display="no" altdistance="0.01" altunitdist="inch" altunit="inch"/>
+<grid distance="0.01" unitdist="inch" unit="inch" style="lines" multiple="1" display="no" altdistance="0.01" altunitdist="inch" altunit="inch"/>
 <layers>
 <layer number="1" name="Top" color="4" fill="1" visible="no" active="no"/>
@@
 <part name="ARR" library="Spade-terminals" deviceset="SPADE-POWER" device=""/>
 <part name="OUT" library="Spade-terminals" deviceset="SPADE-TERMINAL" device="PTH"/>
-<part name="VS_JMP-" library="SparkFun" deviceset="M02" device=""/>
 <part name="CS1" library="Allen" deviceset="S22P015S05" device=""/>
 <part name="C5" library="adafruit" deviceset="C-US" device="C0805" value="0.1uF"/>
@@
 <part name="R13" library="adafruit" deviceset="R-US_" device="R0805" value="100"/>
 <part name="R14" library="adafruit" deviceset="R-US_" device="R0805" value="100"/>
+<part name="JP1" library="SparkFun" deviceset="M01" device="OFFSET" value="M01OFFSET"/>
 </parts>
 <sheets>
@@
 <instance part="ARR" gate="G$1" x="129.794" y="23.114" rot="MR0"/>
 <instance part="OUT" gate="G$1" x="116.586" y="13.208" rot="R180"/>
-<instance part="VS_JMP-" gate="G$1" x="155.702" y="11.176" rot="R90"/>
 <instance part="CS1" gate="G$1" x="66.04" y="142.24" smashed="yes" rot="R270">
 <attribute name="NAME" x="71.12" y="147.32" size="3.81" layer="95" rot="R270"/>
@@
 <instance part="R13" gate="G$1" x="22.86" y="66.04" rot="MR270"/>
 <instance part="R14" gate="G$1" x="22.86" y="127" rot="MR270"/>
+<instance part="JP1" gate="G$1" x="154.94" y="10.16" smashed="yes" rot="R90">
+<attribute name="NAME" x="151.638" y="7.62" size="1.778" layer="95" rot="R90"/>
+</instance>
 </instances>
 <busses>
@@
 <junction x="149.86" y="21.844"/>
 <label x="158.496" y="21.844" size="0.762" layer="95" xref="yes"/>
-<pinref part="VS_JMP-" gate="G$1" pin="2"/>
-<wire x1="153.162" y1="21.844" x2="155.702" y2="21.844" width="0.1524" layer="91"/>
+<wire x1="153.162" y1="21.844" x2="154.94" y2="21.844" width="0.1524" layer="91"/>
+<wire x1="154.94" y1="21.844" x2="155.702" y2="21.844" width="0.1524" layer="91"/>
 <wire x1="155.702" y1="21.844" x2="158.496" y2="21.844" width="0.1524" layer="91"/>
-<wire x1="153.162" y1="18.796" x2="153.162" y2="21.844" width="0.1524" layer="91"/>
-<junction x="153.162" y="21.844"/>
-<pinref part="VS_JMP-" gate="G$1" pin="1"/>
-<wire x1="155.702" y1="18.796" x2="155.702" y2="21.844" width="0.1524" layer="91"/>
-<junction x="155.702" y="21.844"/>
-</segment>
-</net>
+<pinref part="JP1" gate="G$1" pin="1"/>
+<wire x1="154.94" y1="17.78" x2="154.94" y2="21.844" width="0.1524" layer="91"/>
+<junction x="154.94" y="21.844"/>
+</segment>
+</net>
