File: PCB/CMU/Smarttree_CMU_6.sch (EAGLE design)
At the start: 77 parts

Commit message: BMS with the new connectors
Parts:
- removed CMU1, CMU2, CMU3, CMU4: 057-006-0, con-panduit:057-006-0
- removed DEBUG: (no value), SparkFun-Electromechanical:TAC_SWITCHSMD
- removed Q2, Q3, Q5: (no value), adafruit:MOSFET-NREFLOW
- removed R1: 330, adafruit:R-US_M0805
- removed R10, R11, R14: 330, adafruit:R-US_R0805
- removed R15, R16, R17, R18: bypass, adafruit:R-US_M0805
- added 3V3_REG: REG1117, burr-brown:REG1117
- added C7: 0.1uF, SparkFun-Retired:10UF-TANT
- added C8: 10uF, SparkFun-Retired:10UF-TANT
- added CEL1, CEL2, CEL3, CEL4: 8PINCONN, SmartTreeCan:8PINCONN
- added JP1G, JP2G, JP3G, JP4G: JUMPER-SMT_2_NC_TRACE_SILK, SparkFun-Jumpers:JUMPER-SMT_2_NC_TRACE_SILK
- added JP1P, JP2P, JP3P, JP4P: JUMPER-SMT_2_NO_SILK, SparkFun-Jumpers:JUMPER-SMT_2_NO_SILK
- added Q1: (no value), adafruit:MOSFET-NREFLOW
- added U$2, U$3: RELAY-SINGLE_LATCH, SmartTreeCan:RELAY-SINGLE_LATCH
- R5: value 1M -> 330
Connections:
- net !RES_CEL1 renamed !RES_CEL_1&2
- net N$4 renamed SCRN_PWR
- removed net !RES_CEL2: R10.2, U$1.3
- removed net !RES_CEL3: R11.2, U$1.5
- removed net !RES_CEL4: R14.2, U$1.6
- removed net CEL1_GND: CMU1-1.S, Q2.D, R15.2, R5.2
- removed net CEL2_GND: CMU2-1.S, Q3.D, R16.2
- removed net CEL3_GND: CMU3-1.S, Q4.D, R17.2
- removed net CEL4_GND: CMU4-1.S, Q5.D, R18.2
- new net !RES_CEL_3&4: R5.2, U$1.3
- new net N$1: JP1G.1, U$2.P$5
- new net N$10: JP3G.1, U$3.P$5
- new net N$11: JP4G.1, U$3.P$8
- new net N$21: JP2G.1, U$2.P$8
- net 12V: now also 3V3_REG.VIN, C7.+
- net 3.3V: now also 3V3_REG.VOUT, 3V3_REG.VOUT_TAB, C8.+; no longer R1.2, U$1.3V3
- net 5V: now also 5V_REG.VOUT_TAB, JP1P.2, JP2P.2, JP3P.2, JP4P.2, U$2.COIL1, U$2.P$10, U$2.P$3, U$3.COIL1, U$3.P$10, U$3.P$3; no longer R5.1
- net BUTTON: no longer DEBUG.3, DEBUG.4, R1.1
- net CEL1_PWR: now also CEL1.CMU8, JP1P.1, U$2.P$4; no longer CMU1-8.S
- net CEL2_PWR: now also CEL2.CMU8, JP2P.1, U$2.P$9; no longer CMU2-8.S
- net CEL3_PWR: now also CEL3.CMU8, JP3P.1, U$3.P$4; no longer CMU3-8.S
- net CEL4_PWR: now also CEL4.CMU8, JP4P.1, U$3.P$9; no longer CMU4-8.S
- net CSI1: now also CEL1.CMU4; no longer CMU1-4.S
- net CSI2: now also CEL2.CMU4; no longer CMU2-4.S
- net CSI3: now also CEL3.CMU4; no longer CMU3-4.S
- net CSI4: now also CEL4.CMU4; no longer CMU4-4.S
- net CSO1: now also CEL1.CMU2; no longer CMU1-2.S
- net CSO2: now also CEL2.CMU2; no longer CMU2-2.S
- net CSO3: now also CEL3.CMU2; no longer CMU3-2.S
- net CSO4: now also CEL4.CMU2; no longer CMU4-2.S
- net GND: now also 3V3_REG.GND, C7.-, C8.-, CEL1.CMU1, CEL2.CMU1, CEL3.CMU1, CEL4.CMU1, JP1G.2, JP2G.2, JP3G.2, JP4G.2, Q1.S; no longer DEBUG.1, DEBUG.2, Q2.S, Q3.S, Q5.S, R15.1, R16.1, R17.1, R18.1
- net N$3: now also Q4.D, U$2.COIL12; no longer Q3.G, R10.1
- net N$6: now also Q4.G; no longer Q2.G
- net N$7: now also Q1.G, R5.1; no longer Q4.G, R11.1
- net N$9: now also Q1.D, U$3.COIL12; no longer Q5.G, R14.1
- net RI1: now also CEL1.CMU3; no longer CMU1-3.S
- net RI2: now also CEL2.CMU3; no longer CMU2-3.S
- net RI3: now also CEL3.CMU3; no longer CMU3-3.S
- net RI4: now also CEL4.CMU3; no longer CMU4-3.S
- net RO1: now also CEL1.CMU5; no longer CMU1-5.S
- net RO2: now also CEL2.CMU5; no longer CMU2-5.S
- net RO3: now also CEL3.CMU5; no longer CMU3-5.S
- net RO4: now also CEL4.CMU5; no longer CMU4-5.S
- net RX: now also X2.2; no longer X2.3
- net TS1: now also CEL1.CMU6; no longer CMU1-6.S
- net TS2: now also CEL2.CMU6; no longer CMU2-6.S
- net TS3: now also CEL3.CMU6; no longer CMU3-6.S
- net TS4: now also CEL4.CMU6; no longer CMU4-6.S
- net TX: now also X2.3; no longer X2.2
- net VS1: now also CEL1.CMU7; no longer CMU1-7.S
- net VS2: now also CEL2.CMU7; no longer CMU2-7.S
- net VS3: now also CEL3.CMU7; no longer CMU3-7.S
- net VS4: now also CEL4.CMU7; no longer CMU4-7.S
Other:
- note added: "----Schematic ->RS-232 direct mapping (w/o adapter) ->DONE Software reset for each sensor board ->DONE 9 to 3V3 regulator on the board ->DONE get rid of 3v3 ref pin (VREF) ->DONE isolate arduino power"
- note removed: "----Schematic ->RS-232 direct mapping (w/o adapter) ->Software reset for each sensor board ->9 to 3V3 regulator on the board ->get rid of 3v3 ref pin (VREF) ->isolate arduino power"
- moved on the sheet: C10, C6, LED1, LED2, POWER, Q4, R2, R3, R5, R9
