File: PCB/BMS/Smarttree_BMS_6.brd (EAGLE design)
At the start: 90.9 x 58.3 mm, 79 parts

Commit message: holes
Parts:
- moved JP2G 1.61 mm to (68.3, 40.6)
Routing:
- net GND: track 170.8 -> 172.0 mm
Changed lines of the file:
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@@
 <attribute name="NAME" x="13.589" y="20.828" size="0.6096" layer="25" font="vector" ratio="20" rot="R270" align="bottom-center"/>
 </element>
-<element name="JP2G" library="SparkFun-Jumpers" package="SMT-JUMPER_2_NC_TRACE_SILK" value="JUMPER-SMT_2_NC_TRACE_SILK" x="69.85" y="41.148" smashed="yes" rot="R90">
-<attribute name="NAME" x="68.707" y="41.148" size="0.6096" layer="25" font="vector" ratio="20" rot="R90" align="bottom-center"/>
+<element name="JP2G" library="SparkFun-Jumpers" package="SMT-JUMPER_2_NC_TRACE_SILK" value="JUMPER-SMT_2_NC_TRACE_SILK" x="68.326" y="40.64" smashed="yes" rot="R90">
+<attribute name="NAME" x="67.183" y="40.64" size="0.6096" layer="25" font="vector" ratio="20" rot="R90" align="bottom-center"/>
 </element>
 <element name="3V3_REG" library="burr-brown" package="SOT223" value="REG1117" x="22.86" y="36.83" smashed="yes">
@@
 <wire x1="75.946" y1="26.3398" x2="75.946" y2="26.416" width="0.3302" layer="1"/>
 <via x="69.85" y="42.672" extent="1-16" drill="0.3302"/>
-<wire x1="69.85" y1="42.672" x2="69.85" y2="41.656" width="0.3302" layer="1"/>
+<wire x1="69.85" y1="42.672" x2="68.326" y2="41.148" width="0.3302" layer="1"/>
 <via x="16.51" y="35.052" extent="1-16" drill="0.5"/>
 <wire x1="16.002" y1="33.274" x2="16.002" y2="34.544" width="0.3302" layer="1"/>
@@
 <contactref element="U$2" pad="P$8"/>
 <contactref element="JP2G" pad="1"/>
-<wire x1="69.85" y1="39.052" x2="69.85" y2="40.64" width="0.3302" layer="1"/>
+<wire x1="69.85" y1="39.052" x2="68.326" y2="40.132" width="0.3302" layer="1"/>
 </signal>
 <signal name="N$1" class="1">

Commit message: order files
Parts:
- moved JP2P 13.1 mm to (82.8, 43.9)
- moved JP1P 12.9 mm to (80.0, 43.9)
- moved JP1G 1.70 mm to (76.7, 28.4), turned to 90 degrees
- moved X2 1.02 mm to (87.9, 32.3), flipped to the top, turned to 270 degrees
Connections:
- net GND: now also X2.1, X2.6
- net SCRN_PWR: now also X2.7
Routing:
- net GND: track 172.0 -> 472.8 mm, vias 18 -> 17
- net CSI2: track 97.0 -> 45.4 mm, vias 0 -> 1
- net CSI1: track 36.7 -> 72.0 mm, vias 2 -> 3
- net 5V: track 147.9 -> 175.9 mm, vias 2 -> 6
- net VS4: track 117.0 -> 136.3 mm
- net TX: track 61.2 -> 79.8 mm, vias 0 -> 2
- net SCRN_PWR: track 71.9 -> 89.7 mm, vias 1 -> 2
- net TS1OUT: track 8.58 -> 25.1 mm, vias 0 -> 2
- net CSI4: track 105.4 -> 121.5 mm
- net ADDR2: track 24.5 -> 39.3 mm, vias 1 -> 3
- net CEL2_PWR: track 45.9 -> 34.5 mm, vias 2 -> 0
- net CSO3: track 32.5 -> 22.5 mm, vias 3 -> 2
- net CEL1_PWR: track 31.0 -> 21.2 mm, vias 1 -> 0
- net !RES_CEL_1&2: track 46.6 -> 54.9 mm, vias 1 -> 0
- net TX1: track 42.4 -> 49.9 mm
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Other:
- board text removed: "----Layout ->make it nicer ->put analog MUX on the top layer ->make a debugging interface for sensor reading ->switch bypass with jumper -> DONE make sensor board connectors closer to the edge -> add back 5V top and GND bottom planes"

Commit message: aesthetik fixes
Parts:
- removed C10: 0.1uF, SparkFun-Retired:EIA3216
- added C21: 0.1uF, cap-pan40:C-0805
- C7: device SparkFun-Retired:EIA3216 -> cap-pan40:C-0805
- moved C7 7.62 mm to (29.7, 27.9)
Connections:
- net N$24 renamed TS2OUT
- net N$32 renamed TS3OUT
- net N$39 renamed TS4OUT
- net 12V: now also C21.2, C7.2; no longer C10.A, C7.A
- net GND: now also C21.1, C7.1; no longer C10.C, C7.C
Routing:
- net 12V: track 41.4 -> 42.3 mm
- net GND: track 472.8 -> 473.6 mm
Other:
- board text added: "3V3"
- board text added: "5V"
- board text added: "L1"
- board text added: "L2"
- board text removed: "CcA"
Changed lines of the file:
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@@
 <layer number="49" name="Reference" color="7" fill="1" visible="no" active="yes"/>
 <layer number="50" name="dxf" color="7" fill="1" visible="no" active="no"/>
-<layer number="51" name="tDocu" color="7" fill="1" visible="yes" active="yes"/>
+<layer number="51" name="tDocu" color="7" fill="1" visible="no" active="yes"/>
 <layer number="52" name="bDocu" color="7" fill="1" visible="no" active="yes"/>
 <layer number="53" name="tGND_GNDA" color="7" fill="9" visible="no" active="no"/>
@@
 <wire x1="90.932" y1="63.373" x2="0" y2="63.373" width="0" layer="20"/>
 <wire x1="0" y1="63.373" x2="0" y2="5.08" width="0" layer="20"/>
-<text x="42.672" y="6.223" size="0.3048" layer="21">CcA</text>
 <text x="5.08" y="40.64" size="1.778" layer="21" font="vector" rot="R90">SmartTree BMS
 Version 6.0</text>
 <dimension x1="90.932" y1="63.373" x2="0" y2="63.373" x3="45.466" y3="71.12" textsize="1.778" layer="51"/>
 <dimension x1="0" y1="63.373" x2="0" y2="5.08" x3="-12.7" y3="34.2265" textsize="1.778" layer="51"/>
+<text x="20.574" y="36.068" size="1.778" layer="21" font="vector">3V3</text>
+<text x="29.21" y="36.322" size="1.778" layer="21" font="vector">5V</text>
+<text x="87.63" y="7.62" size="1.6764" layer="21" font="vector">L1</text>
+<text x="83.82" y="7.62" size="1.6764" layer="21" font="vector">L2</text>
 </plain>
 <attributes>
@@
 <attribute name="MPN" value="" x="42.418" y="19.431" size="1.778" layer="27" rot="R270" display="off"/>
 </element>
-<element name="C10" library="SparkFun-Retired" package="EIA3216" value="0.1uF" x="29.718" y="27.94" rot="R90">
-<attribute name="PROD_ID" value="CAP-00811" x="29.718" y="27.94" size="1.778" layer="27" rot="R90" display="off"/>
-<attribute name="OC_NEWARK" value="unknown" x="29.718" y="27.94" size="1.778" layer="27" rot="R90" display="off"/>
-<attribute name="MF" value="" x="29.718" y="27.94" size="1.778" layer="27" rot="R90" display="off"/>
-<attribute name="MPN" value="" x="29.718" y="27.94" size="1.778" layer="27" rot="R90" display="off"/>
-</element>
 <element name="C11" library="cap-pan40" package="C-0805" value="" x="38.862" y="19.431" rot="R270">
 <attribute name="OC_NEWARK" value="unknown" x="38.862" y="19.431" size="1.778" layer="27" rot="R270" display="off"/>
@@
 <attribute name="MPN" value="REG1117" x="22.86" y="36.83" size="1.778" layer="27" display="off"/>
 </element>
-<element name="C7" library="SparkFun-Retired" package="EIA3216" value="0.1uF" x="22.098" y="27.94" rot="R90">
-<attribute name="MF" value="" x="22.098" y="27.94" size="1.778" layer="27" rot="R90" display="off"/>
-<attribute name="OC_NEWARK" value="unknown" x="22.098" y="27.94" size="1.778" layer="27" rot="R90" display="off"/>
-<attribute name="PROD_ID" value="CAP-00811" x="22.098" y="27.94" size="1.778" layer="27" rot="R90" display="off"/>
-<attribute name="MPN" value="" x="22.098" y="27.94" size="1.778" layer="27" rot="R90" display="off"/>
-</element>
 <element name="C8" library="SparkFun-Retired" package="EIA3216" value="10uF" x="18.796" y="27.94" rot="R90">
 <attribute name="MF" value="" x="24.13" y="22.098" size="1.778" layer="27" rot="R90" display="off"/>
@@
 <element name="CEL3" library="SmartTreeCan" package="8PINCONN" value="8PINCONN" x="34.798" y="55.88"/>
 <element name="CEL4" library="SmartTreeCan" package="8PINCONN" value="8PINCONN" x="14.478" y="55.88"/>
+<element name="C21" library="cap-pan40" package="C-0805" value="0.1uF" x="22.098" y="27.94" rot="R90">
+<attribute name="MF" value="" x="22.098" y="27.94" size="1.778" layer="27" font="vector" rot="R90" display="off"/>
+<attribute name="MPN" value="" x="22.098" y="27.94" size="1.778" layer="27" font="vector" rot="R90" display="off"/>
+<attribute name="OC_NEWARK" value="unknown" x="22.098" y="27.94" size="1.778" layer="27" font="vector" rot="R90" display="off"/>
+</element>
+<element name="C7" library="cap-pan40" package="C-0805" value="0.1uF" x="29.718" y="27.94" rot="R90">
+<attribute name="MF" value="" x="29.718" y="27.94" size="1.778" layer="27" font="vector" rot="R90" display="off"/>
+<attribute name="MPN" value="" x="29.718" y="27.94" size="1.778" layer="27" font="vector" rot="R90" display="off"/>
+<attribute name="OC_NEWARK" value="unknown" x="29.718" y="27.94" size="1.778" layer="27" font="vector" rot="R90" display="off"/>
+</element>
 </elements>
 <signals>
 <signal name="GND" class="1">
 <contactref element="5V_REG" pad="1"/>
-<contactref element="C10" pad="C"/>
 <contactref element="C6" pad="C"/>
 <contactref element="C4" pad="1"/>
@@
 <contactref element="JP1G" pad="2"/>
 <contactref element="3V3_REG" pad="1"/>
-<contactref element="C7" pad="C"/>
 <contactref element="C8" pad="C"/>
 <contactref element="CEL1" pad="1"/>
@@
 <wire x1="22.0472" y1="26.5811" x2="18.8468" y2="26.5811" width="0.3302" layer="1"/>
 <wire x1="18.8468" y1="26.5811" x2="18.796" y2="26.54" width="0.3302" layer="1"/>
-<wire x1="22.0472" y1="26.5811" x2="22.098" y2="26.54" width="0.3302" layer="1"/>
 <wire x1="23.3807" y1="19.8247" x2="20.8026" y2="19.8247" width="0.3302" layer="1"/>
 <wire x1="26.4033" y1="22.8473" x2="23.3807" y2="19.8247" width="0.3302" layer="1"/>
@@
 <wire x1="26.4033" y1="26.4922" x2="26.416" y2="26.54" width="0.3302" layer="1"/>
 <wire x1="26.5811" y1="26.5811" x2="29.6926" y2="26.5811" width="0.3302" layer="1"/>
-<wire x1="29.6926" y1="26.5811" x2="29.718" y2="26.54" width="0.3302" layer="1"/>
 <wire x1="26.5811" y1="26.5811" x2="26.416" y2="26.54" width="0.3302" layer="1"/>
-<wire x1="26.3144" y1="26.5811" x2="22.225" y2="26.5811" width="0.3302" layer="1"/>
-<wire x1="22.225" y1="26.5811" x2="22.098" y2="26.54" width="0.3302" layer="1"/>
+<wire x1="26.3144" y1="26.5811" x2="22.86" y2="26.5811" width="0.3302" layer="1"/>
+<wire x1="22.86" y1="26.5811" x2="22.225" y2="26.5811" width="0.3302" layer="1"/>
 <wire x1="26.3144" y1="26.5811" x2="26.416" y2="26.54" width="0.3302" layer="1"/>
 <wire x1="28.3591" y1="13.4239" x2="28.3591" y2="11.0236" width="0.3302" layer="1"/>
@@
 <wire x1="29.7815" y1="26.67" x2="29.7815" y2="26.9367" width="0.3302" layer="1"/>
 <wire x1="28.5369" y1="34.0487" x2="28.4734" y2="33.9344" width="0.3302" layer="1"/>
-<wire x1="29.7815" y1="26.67" x2="29.718" y2="26.54" width="0.3302" layer="1"/>
 <wire x1="26.5811" y1="12.8016" x2="26.5811" y2="24.8031" width="0.3302" layer="16"/>
 <wire x1="28.448" y1="10.9347" x2="26.5811" y2="12.8016" width="0.3302" layer="16"/>
@@
 <wire x1="70.104" y1="24.638" x2="69.9643" y2="24.7777" width="0.3302" layer="1"/>
 <wire x1="69.9643" y1="24.7777" x2="68.834" y2="24.7777" width="0.3302" layer="1"/>
+<contactref element="C21" pad="1"/>
+<contactref element="C7" pad="1"/>
+<wire x1="29.7815" y1="26.9367" x2="29.7688" y2="26.9367" width="0.4064" layer="1"/>
+<wire x1="29.7688" y1="26.9367" x2="29.718" y2="26.9875" width="0.4064" layer="1"/>
+<wire x1="22.098" y1="26.9875" x2="22.4536" y2="26.9875" width="0.4064" layer="1"/>
+<wire x1="22.4536" y1="26.9875" x2="22.86" y2="26.5811" width="0.4064" layer="1"/>
+<wire x1="22.225" y1="26.5811" x2="22.0472" y2="26.5811" width="0.4064" layer="1"/>
 </signal>
 <signal name="5V" class="1">
@@
 <signal name="12V" class="1">
 <contactref element="5V_REG" pad="3"/>
-<contactref element="C10" pad="A"/>
 <contactref element="POWER" pad="1"/>
 <contactref element="LED4" pad="A"/>
@@
 <contactref element="F2" pad="2"/>
 <contactref element="3V3_REG" pad="3"/>
-<contactref element="C7" pad="A"/>
 <wire x1="22.1361" y1="30.5816" x2="22.1361" y2="29.4259" width="0.3302" layer="1"/>
 <wire x1="25.1587" y1="33.6042" x2="22.1361" y2="30.5816" width="0.3302" layer="1"/>
-<wire x1="22.1361" y1="29.4259" x2="22.098" y2="29.34" width="0.3302" layer="1"/>
 <wire x1="25.1587" y1="33.6042" x2="25.1714" y2="33.6804" width="0.3302" layer="1"/>
 <wire x1="29.7815" y1="30.6705" x2="29.7815" y2="29.4259" width="0.3302" layer="1"/>
 <wire x1="33.0454" y1="33.9344" x2="29.7815" y2="30.6705" width="0.3302" layer="1"/>
-<wire x1="29.7815" y1="29.4259" x2="29.718" y2="29.34" width="0.3302" layer="1"/>
 <wire x1="26.4922" y1="33.6931" x2="25.3365" y2="33.6931" width="0.3302" layer="1"/>
 <wire x1="29.4259" y1="30.7594" x2="26.4922" y2="33.6931" width="0.3302" layer="1"/>
@@
 <wire x1="15.2908" y1="25.0698" x2="17.78" y2="27.559" width="0.3302" layer="1"/>
 <wire x1="15.2908" y1="22.1361" x2="15.2908" y2="25.0698" width="0.3302" layer="1"/>
-<wire x1="21.9583" y1="29.2481" x2="22.098" y2="29.34" width="0.3302" layer="1"/>
 <wire x1="15.2908" y1="22.1361" x2="15.279" y2="21.971" width="0.3302" layer="1"/>
+<contactref element="C21" pad="2"/>
+<contactref element="C7" pad="2"/>
+<wire x1="29.718" y1="28.8925" x2="29.7815" y2="28.8925" width="0.4064" layer="1"/>
+<wire x1="29.7815" y1="28.8925" x2="29.7815" y2="29.4259" width="0.4064" layer="1"/>
+<wire x1="22.098" y1="28.8925" x2="22.098" y2="29.1084" width="0.4064" layer="1"/>
+<wire x1="22.098" y1="29.1084" x2="21.9583" y2="29.2481" width="0.4064" layer="1"/>
+<wire x1="21.9583" y1="29.2481" x2="22.1361" y2="29.4259" width="0.4064" layer="1"/>
 </signal>
 <signal name="N$13" class="1">
@@
 <via x="44.0944" y="39.7383" extent="1-16" drill="0.3302"/>
 </signal>
-<signal name="N$24">
+<signal name="TS2OUT">
 <contactref element="R21" pad="2"/>
 <contactref element="ANALOG_MUX" pad="5"/>
@@
 <wire x1="31.4706" y1="44.8056" x2="31.398" y2="44.88" width="0.2032" layer="1"/>
 </signal>
-<signal name="N$32">
+<signal name="TS3OUT">
 <contactref element="R25" pad="2"/>
 <contactref element="ANALOG_MUX" pad="23"/>
@@
 <wire x1="51.2953" y1="36.449" x2="51.308" y2="36.3855" width="0.2032" layer="1"/>
 </signal>
-<signal name="N$39">
+<signal name="TS4OUT">
 <contactref element="ANALOG_MUX" pad="19"/>
 <contactref element="R29" pad="2"/>
