File: PCB/BMS/Smarttree_BMS_6.sch (EAGLE design)
At the start: 79 parts

Commit message: order files
Connections:
- net GND: now also X2.1, X2.6
- net SCRN_PWR: now also X2.7
Changed lines of the file:
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@@
 </variantdefs>
 <classes>
-<class number="0" name="default" width="0" drill="0">
+<class number="0" name="default" width="0.2032" drill="0">
 </class>
 <class number="1" name="power" width="0.3302" drill="0">
@@
 <wire x1="154.94" y1="20.32" x2="134.62" y2="20.32" width="0.1524" layer="91"/>
 <junction x="134.62" y="20.32"/>
+<wire x1="154.94" y1="30.48" x2="154.94" y2="43.18" width="0.1524" layer="91"/>
+<junction x="154.94" y="30.48"/>
+<pinref part="X2" gate="G$1" pin="1"/>
+<wire x1="137.16" y1="40.64" x2="137.16" y2="48.26" width="0.1524" layer="91"/>
+<pinref part="X2" gate="G$1" pin="6"/>
+<wire x1="137.16" y1="48.26" x2="152.4" y2="48.26" width="0.1524" layer="91"/>
+<wire x1="152.4" y1="48.26" x2="152.4" y2="43.18" width="0.1524" layer="91"/>
+<wire x1="152.4" y1="43.18" x2="152.4" y2="38.1" width="0.1524" layer="91"/>
+<wire x1="154.94" y1="43.18" x2="152.4" y2="43.18" width="0.1524" layer="91"/>
+<junction x="152.4" y="43.18"/>
 </segment>
 <segment>
@@
 <wire x1="161.798" y1="24.13" x2="161.798" y2="33.02" width="0.1524" layer="91"/>
 <pinref part="X2" gate="G$1" pin="8"/>
-<wire x1="152.4" y1="33.02" x2="161.798" y2="33.02" width="0.1524" layer="91"/>
+<wire x1="152.4" y1="33.02" x2="157.48" y2="33.02" width="0.1524" layer="91"/>
+<wire x1="157.48" y1="33.02" x2="161.798" y2="33.02" width="0.1524" layer="91"/>
 <wire x1="161.798" y1="33.02" x2="162.56" y2="33.02" width="0.1524" layer="91"/>
 <junction x="161.798" y="33.02"/>
 <label x="139.446" y="24.13" size="1.778" layer="95"/>
-</segment>
-</net>
+<pinref part="X2" gate="G$1" pin="7"/>
+<wire x1="152.4" y1="35.56" x2="157.48" y2="35.56" width="0.1524" layer="91"/>
+<wire x1="157.48" y1="35.56" x2="157.48" y2="33.02" width="0.1524" layer="91"/>
+<junction x="157.48" y="33.02"/>
+</segment>
+</net>

Commit message: aesthetik fixes
Parts:
- removed C10: 0.1uF, SparkFun-Retired:10UF-TANT
- added C21: 0.1uF, cap-pan40:C-NP-SMD-0805
- C7: device SparkFun-Retired:10UF-TANT -> cap-pan40:C-NP-SMD-0805
Connections:
- net N$24 renamed TS2OUT
- net N$32 renamed TS3OUT
- net N$39 renamed TS4OUT
- net 12V: now also C21.2, C7.2; no longer C10.+, C7.+
- net GND: now also C21.1, C7.1; no longer C10.-, C7.-
Other:
- note removed: "----Schematic ->RS-232 direct mapping (w/o adapter) ->DONE Software reset for each sensor board ->DONE 9 to 3V3 regulator on the board ->DONE get rid of 3v3 ref pin (VREF) ->DONE isolate arduino power"
Changed lines of the file:
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@@
 <part name="SUPPLY10" library="eagle-book" deviceset="GND" device=""/>
 <part name="5V_REG" library="burr-brown" deviceset="REG1117" device=""/>
-<part name="C10" library="SparkFun-Retired" deviceset="10UF-TANT" device="" value="0.1uF">
-<attribute name="MF" value=""/>
-<attribute name="MPN" value=""/>
-<attribute name="OC_NEWARK" value="unknown"/>
-</part>
 <part name="C6" library="SparkFun-Retired" deviceset="10UF-TANT" device="" value="10uF">
 <attribute name="MF" value=""/>
@@
 <part name="SUPPLY5" library="eagle-book" deviceset="GND" device=""/>
 <part name="3V3_REG" library="burr-brown" deviceset="REG1117" device=""/>
-<part name="C7" library="SparkFun-Retired" deviceset="10UF-TANT" device="" value="0.1uF">
-<attribute name="MF" value=""/>
-<attribute name="MPN" value=""/>
-<attribute name="OC_NEWARK" value="unknown"/>
-</part>
 <part name="C8" library="SparkFun-Retired" deviceset="10UF-TANT" device="" value="10uF">
 <attribute name="MF" value=""/>
@@
 <part name="CEL3" library="SmartTreeCan" deviceset="8PINCONN" device=""/>
 <part name="CEL4" library="SmartTreeCan" deviceset="8PINCONN" device=""/>
+<part name="C21" library="cap-pan40" deviceset="C-NP" device="-SMD-0805" value="0.1uF">
+<attribute name="MF" value=""/>
+<attribute name="MPN" value=""/>
+<attribute name="OC_NEWARK" value="unknown"/>
+</part>
+<part name="C7" library="cap-pan40" deviceset="C-NP" device="-SMD-0805" value="0.1uF">
+<attribute name="MF" value=""/>
+<attribute name="MPN" value=""/>
+<attribute name="OC_NEWARK" value="unknown"/>
+</part>
 </parts>
 <sheets>
 <sheet>
 <plain>
-<text x="177.8" y="22.86" size="6.4516" layer="91">BMS and Power</text>
-<text x="12.7" y="152.4" size="1.778" layer="97">----Schematic
--&gt;RS-232 direct mapping (w/o adapter)
--&gt;DONE Software reset for each sensor board
--&gt;DONE 9 to 3V3 regulator on the board
--&gt;DONE get rid of 3v3 ref pin (VREF)
--&gt;DONE isolate arduino power</text>
+<text x="177.8" y="22.86" size="6.4516" layer="91" font="vector">BMS and Power</text>
 <wire x1="144.78" y1="172.72" x2="144.78" y2="99.06" width="0.1524" layer="97"/>
 <wire x1="144.78" y1="99.06" x2="254" y2="99.06" width="0.1524" layer="97"/>
@@
 <instance part="SUPPLY10" gate="GND" x="86.36" y="119.38"/>
 <instance part="5V_REG" gate="G$1" x="210.82" y="83.82"/>
-<instance part="C10" gate="G$1" x="193.04" y="76.2">
-<attribute name="OC_NEWARK" x="193.04" y="76.2" size="1.778" layer="96" display="off"/>
-<attribute name="MF" x="193.04" y="76.2" size="1.778" layer="96" display="off"/>
-<attribute name="MPN" x="193.04" y="76.2" size="1.778" layer="96" display="off"/>
-</instance>
 <instance part="C6" gate="G$1" x="226.06" y="76.2">
 <attribute name="OC_NEWARK" x="226.06" y="76.2" size="1.778" layer="96" display="off"/>
@@
 <instance part="SUPPLY5" gate="GND" x="167.64" y="60.96"/>
 <instance part="3V3_REG" gate="G$1" x="167.64" y="83.82"/>
-<instance part="C7" gate="G$1" x="149.86" y="76.2">
-<attribute name="OC_NEWARK" x="149.86" y="76.2" size="1.778" layer="96" display="off"/>
-<attribute name="MF" x="149.86" y="76.2" size="1.778" layer="96" display="off"/>
-<attribute name="MPN" x="149.86" y="76.2" size="1.778" layer="96" display="off"/>
-</instance>
 <instance part="C8" gate="G$1" x="182.88" y="76.2">
 <attribute name="OC_NEWARK" x="182.88" y="76.2" size="1.778" layer="96" display="off"/>
@@
 </instance>
 <instance part="SUPPLY20" gate="G$1" x="182.88" y="88.9"/>
+<instance part="C21" gate="G$1" x="149.86" y="76.2" rot="R90">
+<attribute name="OC_NEWARK" x="149.86" y="76.2" size="1.778" layer="96" display="off"/>
+<attribute name="MF" x="149.86" y="76.2" size="1.778" layer="96" display="off"/>
+<attribute name="MPN" x="149.86" y="76.2" size="1.778" layer="96" display="off"/>
+</instance>
+<instance part="C7" gate="G$1" x="193.04" y="76.2" rot="R90">
+<attribute name="OC_NEWARK" x="193.04" y="76.2" size="1.778" layer="96" display="off"/>
+<attribute name="MF" x="193.04" y="76.2" size="1.778" layer="96" display="off"/>
+<attribute name="MPN" x="193.04" y="76.2" size="1.778" layer="96" display="off"/>
+</instance>
 </instances>
 <busses>
@@
 <pinref part="SUPPLY19" gate="GND" pin="GND"/>
 <wire x1="210.82" y1="68.58" x2="210.82" y2="63.5" width="0.1524" layer="91"/>
-<pinref part="C10" gate="G$1" pin="-"/>
-<wire x1="193.04" y1="68.58" x2="193.04" y2="71.12" width="0.1524" layer="91"/>
+<wire x1="193.04" y1="68.58" x2="193.04" y2="73.66" width="0.1524" layer="91"/>
 <pinref part="C6" gate="G$1" pin="-"/>
 <wire x1="226.06" y1="68.58" x2="226.06" y2="71.12" width="0.1524" layer="91"/>
+<pinref part="C7" gate="G$1" pin="1"/>
 </segment>
 <segment>
@@
 <pinref part="SUPPLY5" gate="GND" pin="GND"/>
 <wire x1="167.64" y1="68.58" x2="167.64" y2="63.5" width="0.1524" layer="91"/>
-<pinref part="C7" gate="G$1" pin="-"/>
-<wire x1="149.86" y1="68.58" x2="149.86" y2="71.12" width="0.1524" layer="91"/>
+<wire x1="149.86" y1="68.58" x2="149.86" y2="73.66" width="0.1524" layer="91"/>
 <pinref part="C8" gate="G$1" pin="-"/>
 <wire x1="182.88" y1="68.58" x2="182.88" y2="71.12" width="0.1524" layer="91"/>
+<pinref part="C21" gate="G$1" pin="1"/>
 </segment>
 </net>
@@
 <pinref part="5V_REG" gate="G$1" pin="VIN"/>
 <wire x1="198.12" y1="83.82" x2="193.04" y2="83.82" width="0.1524" layer="91"/>
-<pinref part="C10" gate="G$1" pin="+"/>
 <wire x1="193.04" y1="78.74" x2="193.04" y2="83.82" width="0.1524" layer="91"/>
 <junction x="193.04" y="83.82"/>
+<pinref part="C7" gate="G$1" pin="2"/>
 </segment>
 <segment>
@@
 <pinref part="3V3_REG" gate="G$1" pin="VIN"/>
 <wire x1="154.94" y1="83.82" x2="149.86" y2="83.82" width="0.1524" layer="91"/>
-<pinref part="C7" gate="G$1" pin="+"/>
 <wire x1="149.86" y1="78.74" x2="149.86" y2="83.82" width="0.1524" layer="91"/>
 <junction x="149.86" y="83.82"/>
+<pinref part="C21" gate="G$1" pin="2"/>
 </segment>
 </net>
@@
 <sheet>
 <plain>
-<text x="172.72" y="25.4" size="6.096" layer="91">Sensor and Connector</text>
+<text x="172.72" y="25.4" size="4.318" layer="91" font="vector">Sensor and Connector</text>
 </plain>
 <instances>
@@
 </segment>
 </net>
-<net name="N$24" class="0">
+<net name="TS2OUT" class="0">
 <segment>
 <pinref part="R21" gate="G$1" pin="2"/>
@@
 <wire x1="35.56" y1="137.16" x2="68.58" y2="137.16" width="0.1524" layer="91"/>
 <junction x="35.56" y="137.16"/>
+<label x="38.1" y="137.16" size="1.778" layer="95"/>
 </segment>
 </net>
@@
 </segment>
 </net>
-<net name="N$32" class="0">
+<net name="TS3OUT" class="0">
 <segment>
 <pinref part="R25" gate="G$1" pin="2"/>
@@
 <pinref part="C12" gate="G$1" pin="2"/>
 <junction x="35.56" y="106.68"/>
+<label x="38.1" y="106.68" size="1.778" layer="95"/>
 </segment>
 </net>
@@
 </segment>
 </net>
-<net name="N$39" class="0">
+<net name="TS4OUT" class="0">
 <segment>
 <pinref part="ANALOG_MUX" gate="G$1" pin="CHAN12"/>
@@
 <wire x1="35.56" y1="76.2" x2="33.02" y2="76.2" width="0.1524" layer="91"/>
 <junction x="35.56" y="76.2"/>
+<label x="38.1" y="76.2" size="1.778" layer="95"/>
 </segment>
 </net>
@@
 <wire x1="45.72" y1="167.64" x2="45.72" y2="170.18" width="0.1524" layer="91"/>
 <junction x="45.72" y="170.18"/>
+<label x="33.02" y="170.18" size="1.778" layer="95"/>
 </segment>
 </net>
@@
 </schematic>
 </drawing>
-<compatibility>
-<note version="6.3" minversion="6.2.2" severity="warning">
-Since Version 6.2.2 text objects can contain more than one line,
-which will not be processed correctly with this version.
-</note>
-</compatibility>
 </eagle>
